File: qspimux2/qspimux.kicad_pcb (KiCad board)
At the start: 4 copper layers, 14.2 x 23.2 mm, 13 parts, among them J101 Conn_01x10_MountingPin, J102 Conn_02x04_Odd_Even, J103 Conn_02x04_Odd_Even, U101 TS3A27518ERTWR, U102 MAX40200AUK, U103 MAX40200AUK

Commit message: fix wrong signal name
the connection was right, but the name had an off-by-one
Connections:
- net /IO0_DO_BOARD renamed /IO1_DO_BOARD
